File: hardware/schematic-OLED_SPI.sch (KiCad schematic (older format))
At the start: 12 parts

Commit message: Updated schematic on missing GND for buttons
Connections:
- net GND: now also button_1.1, button_2.1, button_3.1
- net at U?.2 (VDD_out): now also NA.2 (VCC)
- net at U?.4 (P1.00): now also U?.1
- net at U?.8 (P1.13): now also NA.4 (SDA)
Changed lines of the file:
@@
 	7737 5623 8937 5623
 Wire Notes Line
-	8937 5623 8937 7223
-Wire Notes Line
-	8937 7223 7737 7223
+	8937 5623 8937 7348
+Wire Notes Line
+	8937 7348 7737 7348
 Text Notes 7737 5573 0    79   ~ 0
 850C remote keypad
@@
 TSDZ2_5V
 Wire Notes Line
-	7737 5623 7737 7223
+	7737 5623 7737 7348
 $Comp
 L Wired_remote:Switch_SW_Push button_3
@@
 Wire Wire Line
 	13198 4432 13326 4432
+Wire Wire Line
+	10296 5364 9910 5364
+Wire Wire Line
+	9910 5364 9910 6790
+Wire Wire Line
+	9910 6790 8780 6790
+Wire Wire Line
+	8780 6790 8780 7200
+Wire Wire Line
+	8780 7200 7956 7200
+Wire Wire Line
+	7956 7200 7956 7074
+Connection ~ 10296 5364
+Connection ~ 7956 7074
 $EndSCHEMATC
